Commit message: directory restructure and readme update

File: src/sim_mdrs/urdf/gazebo.urdf.xacro (robot description, xacro)
@@ -113,5 +113,5 @@
   <gazebo>
     <plugin filename="libgazebo_ros2_control.so" name="gazebo_ros2_control">
-      <parameters>$(find rpi_MDRS)/config/controller_velocity.yaml</parameters>
+      <parameters>$(find sim_mdrs)/config/controller_velocity.yaml</parameters>
     </plugin>
   </gazebo>

File: src/sim_mdrs/urdf/osr.urdf.xacro (robot description, xacro)
@@ -16,6 +16,6 @@
       <color rgba="0.5451 0.2706 0.0745 1"/>
     </material>
-    <xacro:include filename="$(find rpi_MDRS)/urdf/gazebo.urdf.xacro"/>
-    <xacro:include filename="$(find rpi_MDRS)/urdf/insert_transmission.urdf.xacro"/>
+    <xacro:include filename="$(find sim_mdrs)/urdf/gazebo.urdf.xacro"/>
+    <xacro:include filename="$(find sim_mdrs)/urdf/insert_transmission.urdf.xacro"/>
     <link name="base_footprint"/>
     <link name="base_link">
@@ -23,5 +23,5 @@
             <origin rpy="0 0 0" xyz="0 0 0.0"/>
             <geometry>
-                <mesh filename="file://$(find rpi_MDRS)/urdf/meshes/body.stl"/>
+                <mesh filename="file://$(find sim_mdrs)/urdf/meshes/body.stl"/>
             </geometry>
         </collision>
@@ -29,5 +29,5 @@
             <origin rpy="0 0 0" xyz="0 0 0.0"/>
             <geometry>
-                <mesh filename="file://$(find rpi_MDRS)/urdf/meshes/body.stl"/>
+                <mesh filename="file://$(find sim_mdrs)/urdf/meshes/body.stl"/>
             </geometry>
             <material name="brown"/>
@@ -49,5 +49,5 @@
             <origin rpy="0 0 -3.14" xyz="0 0 0.0"/>
             <geometry>
-                <mesh filename="file://$(find rpi_MDRS)/urdf/meshes/box_link.stl"/>
+                <mesh filename="file://$(find sim_mdrs)/urdf/meshes/box_link.stl"/>
             </geometry>
         </collision>
@@ -55,5 +55,5 @@
             <origin rpy="0 0 -3.14" xyz="0 0 0"/>
             <geometry>
-                <mesh filename="file://$(find rpi_MDRS)/urdf/meshes/box_link.stl"/>
+                <mesh filename="file://$(find sim_mdrs)/urdf/meshes/box_link.stl"/>
             </geometry>
             <material name="silver"/>
@@ -76,5 +76,5 @@
                 <origin rpy="0 0.2 0" xyz="0 0 0"/>
                 <geometry>
-                    <mesh filename="file://$(find rpi_MDRS)/urdf/meshes/arm.stl"/>
+                    <mesh filename="file://$(find sim_mdrs)/urdf/meshes/arm.stl"/>
                 </geometry>
             </collision>
@@ -82,5 +82,5 @@
                 <origin rpy="0 0.2 0" xyz="0 0 0"/>
                 <geometry>
-                    <mesh filename="file://$(find rpi_MDRS)/urdf/meshes/arm.stl"/>
+                    <mesh filename="file://$(find sim_mdrs)/urdf/meshes/arm.stl"/>
                 </geometry>
                 <material name="silver"/>
@@ -106,5 +106,5 @@
                 <origin rpy="0 0 ${origin}" xyz="0 0 0.0"/>
                 <geometry>
-                    <mesh filename="file://$(find rpi_MDRS)/urdf/meshes/turn_${prefix}.stl"/>
+                    <mesh filename="file://$(find sim_mdrs)/urdf/meshes/turn_${prefix}.stl"/>
                 </geometry>
             </collision>
@@ -112,5 +112,5 @@
                 <origin rpy="0 0 ${origin}" xyz="0 0 0.0"/>
                 <geometry>
-                    <mesh filename="file://$(find rpi_MDRS)/urdf/meshes/turn_${prefix}.stl"/>
+                    <mesh filename="file://$(find sim_mdrs)/urdf/meshes/turn_${prefix}.stl"/>
                 </geometry>
                 <material name="silver"/>
@@ -136,5 +136,5 @@
                 <origin rpy="0 0 1.57" xyz="0 0 0.0"/>
                 <geometry>
-                    <mesh filename="file://$(find rpi_MDRS)/urdf/meshes/body_axis.stl"/>
+                    <mesh filename="file://$(find sim_mdrs)/urdf/meshes/body_axis.stl"/>
                 </geometry>
             </collision>
@@ -142,5 +142,5 @@
                 <origin rpy="0 0 1.57" xyz="0 0 0.0"/>
                 <geometry>
-                    <mesh filename="file://$(find rpi_MDRS)/urdf/meshes/body_axis.stl"/>
+                    <mesh filename="file://$(find sim_mdrs)/urdf/meshes/body_axis.stl"/>
                 </geometry>
                 <material name="silver"/>
@@ -166,11 +166,11 @@
                 <origin rpy="0 0 0" xyz="0 0 0.0"/>
                 <geometry>
-                    <mesh filename="file://$(find rpi_MDRS)/urdf/meshes/rockerbogie_middle_1.stl"/>
-                </geometry>
-            </collision>
-            <visual>
-                <origin rpy="0 0 0" xyz="0 0 0.0"/>
-                <geometry>
-                    <mesh filename="file://$(find rpi_MDRS)/urdf/meshes/rockerbogie_middle_1.stl"/>
+                    <mesh filename="file://$(find sim_mdrs)/urdf/meshes/rockerbogie_middle_1.stl"/>
+                </geometry>
+            </collision>
+            <visual>
+                <origin rpy="0 0 0" xyz="0 0 0.0"/>
+                <geometry>
+                    <mesh filename="file://$(find sim_mdrs)/urdf/meshes/rockerbogie_middle_1.stl"/>
                 </geometry>
                 <material name="silver"/>
@@ -193,11 +193,11 @@
                 <origin rpy="0 0 0" xyz="0 0 0.0"/>
                 <geometry>
-                    <mesh filename="file://$(find rpi_MDRS)/urdf/meshes/rockerbogie_front_1.stl"/>
-                </geometry>
-            </collision>
-            <visual>
-                <origin rpy="0 0 0" xyz="0 0 0.0"/>
-                <geometry>
-                    <mesh filename="file://$(find rpi_MDRS)/urdf/meshes/rockerbogie_front_1.stl"/>
+                    <mesh filename="file://$(find sim_mdrs)/urdf/meshes/rockerbogie_front_1.stl"/>
+                </geometry>
+            </collision>
+            <visual>
+                <origin rpy="0 0 0" xyz="0 0 0.0"/>
+                <geometry>
+                    <mesh filename="file://$(find sim_mdrs)/urdf/meshes/rockerbogie_front_1.stl"/>
                 </geometry>
                 <material name="silver"/>
@@ -224,5 +224,5 @@
                 <origin rpy="0 0 ${dir*-1.57}" xyz="0 0 0.0"/>
                 <geometry>
-                    <mesh filename="file://$(find rpi_MDRS)/urdf/meshes/wheel_link_left_2.stl"/>
+                    <mesh filename="file://$(find sim_mdrs)/urdf/meshes/wheel_link_left_2.stl"/>
                 </geometry>
             </collision>
@@ -230,5 +230,5 @@
                 <origin rpy="0 0 ${dir*-1.57}" xyz="0 0 0.0"/>
                 <geometry>
-                    <mesh filename="file://$(find rpi_MDRS)/urdf/meshes/wheel_link_left_2.stl"/>
+                    <mesh filename="file://$(find sim_mdrs)/urdf/meshes/wheel_link_left_2.stl"/>
                 </geometry>
                 <material name="silver"/>
@@ -252,5 +252,5 @@
                 <origin rpy="${origin} 0 ${-dir*1.57}" xyz="0 0 0.0"/>
                 <geometry>
-                    <mesh filename="file://$(find rpi_MDRS)/urdf/meshes/wheel_middle_left.stl"/>
+                    <mesh filename="file://$(find sim_mdrs)/urdf/meshes/wheel_middle_left.stl"/>
                 </geometry>
             </collision>
@@ -258,5 +258,5 @@
                 <origin rpy="${origin} 0 ${-dir*1.57}" xyz="0 0 0.0"/>
                 <geometry>
-                    <mesh filename="file://$(find rpi_MDRS)/urdf/meshes/wheel_middle_left.stl"/>
+                    <mesh filename="file://$(find sim_mdrs)/urdf/meshes/wheel_middle_left.stl"/>
                 </geometry>
                 <material name="silver"/>
@@ -278,5 +278,5 @@
                 <origin rpy="0 0 ${-dir*1.57}" xyz="0 0 0.0"/>
                 <geometry>
-                    <mesh filename="file://$(find rpi_MDRS)/urdf/meshes/wheel_link_left_2.stl"/>
+                    <mesh filename="file://$(find sim_mdrs)/urdf/meshes/wheel_link_left_2.stl"/>
                 </geometry>
             </collision>
@@ -284,5 +284,5 @@
                 <origin rpy="0 0 ${-dir*1.57}" xyz="0 0 0.0"/>
                 <geometry>
-                    <mesh filename="file://$(find rpi_MDRS)/urdf/meshes/wheel_link_left_2.stl"/>
+                    <mesh filename="file://$(find sim_mdrs)/urdf/meshes/wheel_link_left_2.stl"/>
                 </geometry>
                 <material name="silver"/>
@@ -310,5 +310,5 @@
                 <origin rpy="-1.57 0 ${origin}" xyz="0 0 0.0"/>
                 <geometry>
-                    <mesh filename="file://$(find rpi_MDRS)/urdf/meshes/wheel.stl"/>
+                    <mesh filename="file://$(find sim_mdrs)/urdf/meshes/wheel.stl"/>
                 </geometry>
                 <surface>
@@ -324,5 +324,5 @@
                 <origin rpy="-1.57 0 ${origin}" xyz="0 0 0.0"/>
                 <geometry>
-                    <mesh filename="file://$(find rpi_MDRS)/urdf/meshes/wheel.stl"/>
+                    <mesh filename="file://$(find sim_mdrs)/urdf/meshes/wheel.stl"/>
                 </geometry>
                 <material name="black"/>
@@ -345,5 +345,5 @@
                 <origin rpy="-1.57 0 ${origin}" xyz="0 0 0.0"/>
                 <geometry>
-                    <mesh filename="file://$(find rpi_MDRS)/urdf/meshes/wheel.stl"/>
+                    <mesh filename="file://$(find sim_mdrs)/urdf/meshes/wheel.stl"/>
                 </geometry>
                 <surface>
@@ -359,5 +359,5 @@
                 <origin rpy="-1.57 0 ${origin}" xyz="0 0 0.0"/>
                 <geometry>
-                    <mesh filename="file://$(find rpi_MDRS)/urdf/meshes/wheel.stl"/>
+                    <mesh filename="file://$(find sim_mdrs)/urdf/meshes/wheel.stl"/>
                 </geometry>
                 <material name="black"/>
@@ -380,5 +380,5 @@
                 <origin rpy="-1.57 0 ${origin}" xyz="0 0 0.0"/>
                 <geometry>
-                    <mesh filename="file://$(find rpi_MDRS)/urdf/meshes/wheel.stl"/>
+                    <mesh filename="file://$(find sim_mdrs)/urdf/meshes/wheel.stl"/>
                 </geometry>
                 <surface>
@@ -394,5 +394,5 @@
                 <origin rpy="-1.57 0 ${origin}" xyz="0 0 0.0"/>
                 <geometry>
-                    <mesh filename="file://$(find rpi_MDRS)/urdf/meshes/wheel.stl"/>
+                    <mesh filename="file://$(find sim_mdrs)/urdf/meshes/wheel.stl"/>
                 </geometry>
                 <material name="black"/>
