Commit message: changed fourth_link by arm_link and checked rotation axis

File: src/sim_mdrs/urdf/arm.urdf.xacro (robot description, xacro)
@@ -39,5 +39,5 @@
     <child link="second_link"/>
     <origin xyz="0 0 ${second_link_length / 2}" rpy="0 0 0"/>
-    <axis xyz="0 0 1"/>
+    <axis xyz="1 0 0"/>
     <limit lower="-1.57" upper="1.57" effort="10" velocity="1"/>
   </joint>
@@ -54,5 +54,5 @@
     <child link="third_link"/>
     <origin xyz="0 0 ${third_link_length / 2}" rpy="0 0 0"/>
-    <axis xyz="0 0 1"/>
+    <axis xyz="1 0 0"/>
     <limit lower="-1.57" upper="1.57" effort="10" velocity="1"/>
   </joint>
@@ -67,7 +67,7 @@
 <joint name="joint4" type="revolute">
     <parent link="third_link"/>
-    <child link="fourth_link"/>
+    <child link="arm_link"/>
     <origin xyz="0 0 ${base_link_length / 2}" rpy="0 0 0"/>
-    <axis xyz="0 0 1"/>
+    <axis xyz="1 0 0"/>
     <limit lower="-1.57" upper="1.57" effort="10" velocity="1"/>
   </joint>
@@ -94,5 +94,5 @@
   </link>
   <joint name="gripper_joint" type="fixed">
-    <parent link="fourth_link"/>
+    <parent link="arm_link"/>
     <child link="gripper_base"/>
     <origin xyz="0 0 ${fourth_link_length / 2}" rpy="0 0 0"/>

Commit message: setting up gazebo for arm simulation

File: src/sim_mdrs/urdf/arm.urdf.xacro (robot description, xacro)
@@ -1,4 +1,7 @@
 <?xml version="1.0"?>
 <robot xmlns:xacro="http://www.ros.org/wiki/xacro" name="my_robot_arm">
+  <plugin name="gazebo_ros_control" filename="libgazebo_ros_control.so">
+    <robotNamespace>/</robotNamespace>
+  </plugin>
   <!-- Properties -->
   <xacro:property name="base_link_length" value="0.5"/>
@@ -9,4 +12,16 @@
   <xacro:property name="gripper_length" value="1.0"/>
   <xacro:property name="link_radius" value="0.05"/>
+  <xacro:macro name="define_materials" params="">
+    <material name="blue">
+      <color rgba="0.0 0.0 1.0 1.0"/>
+    </material>
+    <material name="red">
+      <color rgba="1.0 0.0 0.0 1.0"/>
+    </material>
+    <material name="gray">
+      <color rgba="0.5 0.5 0.5 1.0"/>
+    </material>
+  </xacro:macro>
+  <xacro:define_materials/>
   <!-- Base Link -->
   <link name="base_link">
@@ -15,16 +30,18 @@
         <cylinder length="${base_link_length}" radius="${link_radius}"/>
       </geometry>
-      <material name="blue"/>
+      <material name="gray"/>
     </visual>
+    <collision>
+      <geometry>
+        <cylinder length="${base_link_length}" radius="${link_radius}"/>
+      </geometry>
+    </collision>
+    <inertial>
+      <mass value="1.0"/>
+      <origin xyz="0 0 0"/>
+      <inertia ixx="0.01" ixy="0.0" ixz="0.0" iyy="0.01" iyz="0.0" izz="0.01"/>
+    </inertial>
   </link>
-  <!-- Joint 1 -->
-  <joint name="joint1" type="revolute">
-    <parent link="base_link"/>
-    <child link="first_link"/>
-    <origin xyz="0 0 ${base_link_length / 2}" rpy="0 0 0"/>
-    <axis xyz="0 0 1"/>
-    <limit lower="-1.57" upper="1.57" effort="10" velocity="1"/>
-  </joint>
-  <!-- Arm Link -->
+  <!-- First Link -->
   <link name="first_link">
     <visual>
@@ -32,14 +49,18 @@
         <cylinder length="${first_link_length}" radius="${link_radius}"/>
       </geometry>
-      <material name="red"/>
+      <material name="blue"/>
     </visual>
+    <collision>
+      <geometry>
+        <cylinder length="${first_link_length}" radius="${link_radius}"/>
+      </geometry>
+    </collision>
+    <inertial>
+      <mass value="0.5"/>
+      <origin xyz="0 0 0"/>
+      <inertia ixx="0.005" ixy="0.0" ixz="0.0" iyy="0.005" iyz="0.0" izz="0.005"/>
+    </inertial>
   </link>
-<joint name="joint2" type="revolute">
-    <parent link="first_link"/>
-    <child link="second_link"/>
-    <origin xyz="0 0 ${second_link_length / 2}" rpy="0 0 0"/>
-    <axis xyz="0 0 1"/>
-    <limit lower="-1.57" upper="1.57" effort="10" velocity="1"/>
-  </joint>
+  <!-- Second Link -->
   <link name="second_link">
     <visual>
@@ -49,12 +70,16 @@
       <material name="red"/>
     </visual>
+    <collision>
+      <geometry>
+        <cylinder length="${second_link_length}" radius="${link_radius}"/>
+      </geometry>
+    </collision>
+    <inertial>
+      <mass value="0.5"/>
+      <origin xyz="0 0 0"/>
+      <inertia ixx="0.005" ixy="0.0" ixz="0.0" iyy="0.005" iyz="0.0" izz="0.005"/>
+    </inertial>
   </link>
-<joint name="joint3" type="revolute">
-    <parent link="second_link"/>
-    <child link="third_link"/>
-    <origin xyz="0 0 ${third_link_length / 2}" rpy="0 0 0"/>
-    <axis xyz="0 0 1"/>
-    <limit lower="-1.57" upper="1.57" effort="10" velocity="1"/>
-  </joint>
+  <!-- Third Link -->
   <link name="third_link">
     <visual>
@@ -62,15 +87,19 @@
         <cylinder length="${third_link_length}" radius="${link_radius}"/>
       </geometry>
-      <material name="red"/>
+      <material name="blue"/>
     </visual>
+    <collision>
+      <geometry>
+        <cylinder length="${third_link_length}" radius="${link_radius}"/>
+      </geometry>
+    </collision>
+    <inertial>
+      <mass value="0.5"/>
+      <origin xyz="0 0 0"/>
+      <inertia ixx="0.005" ixy="0.0" ixz="0.0" iyy="0.005" iyz="0.0" izz="0.005"/>
+    </inertial>
   </link>
-<joint name="joint4" type="revolute">
-    <parent link="third_link"/>
-    <child link="fourth_link"/>
-    <origin xyz="0 0 ${base_link_length / 2}" rpy="0 0 0"/>
-    <axis xyz="0 0 1"/>
-    <limit lower="-1.57" upper="1.57" effort="10" velocity="1"/>
-  </joint>
-  <link name="arm_link">
+  <!-- Fourth Link -->
+  <link name="fourth_link">
     <visual>
       <geometry>
@@ -79,54 +108,69 @@
       <material name="red"/>
     </visual>
+    <collision>
+      <geometry>
+        <cylinder length="${fourth_link_length}" radius="${link_radius}"/>
+      </geometry>
+    </collision>
+    <inertial>
+      <mass value="0.8"/>
+      <origin xyz="0 0 0"/>
+      <inertia ixx="0.01" ixy="0.0" ixz="0.0" iyy="0.01" iyz="0.0" izz="0.01"/>
+    </inertial>
   </link>
-  <!-- Gripper Properties -->
-  <xacro:property name="gripper_finger_length" value="0.1"/>
-  <xacro:property name="gripper_finger_width" value="0.02"/>
-  <xacro:property name="gripper_finger_range" value="0.04"/>
-  <!-- Gripper Base -->
-  <link name="gripper_base">
+  <!-- Gripper Link -->
+  <link name="gripper">
     <visual>
       <geometry>
-        <box size="0.1 0.1 0.02"/>
+        <cylinder length="${gripper_length}" radius="${link_radius}"/>
       </geometry>
       <material name="gray"/>
     </visual>
+    <collision>
+      <geometry>
+        <cylinder length="${gripper_length}" radius="${link_radius}"/>
+      </geometry>
+    </collision>
+    <inertial>
+      <mass value="0.3"/>
+      <origin xyz="0 0 0"/>
+      <inertia ixx="0.002" ixy="0.0" ixz="0.0" iyy="0.002" iyz="0.0" izz="0.002"/>
+    </inertial>
   </link>
-  <joint name="gripper_joint" type="fixed">
+  <!-- Joints -->
+  <joint name="joint1" type="revolute">
+    <parent link="base_link"/>
+    <child link="first_link"/>
+    <origin xyz="0 0 ${base_link_length/2}" rpy="0 0 0"/>
+    <axis xyz="0 1 0"/>
+    <limit effort="10.0" velocity="1.0" lower="-1.57" upper="1.57"/>
+  </joint>
+  <joint name="joint2" type="revolute">
+    <parent link="first_link"/>
+    <child link="second_link"/>
+    <origin xyz="0 0 ${first_link_length/2}" rpy="0 0 0"/>
+    <axis xyz="0 1 0"/>
+    <limit effort="10.0" velocity="1.0" lower="-1.57" upper="1.57"/>
+  </joint>
+  <joint name="joint3" type="revolute">
+    <parent link="second_link"/>
+    <child link="third_link"/>
+    <origin xyz="0 0 ${second_link_length/2}" rpy="0 0 0"/>
+    <axis xyz="0 1 0"/>
+    <limit effort="10.0" velocity="1.0" lower="-1.57" upper="1.57"/>
+  </joint>
+  <joint name="joint4" type="revolute">
+    <parent link="third_link"/>
+    <child link="fourth_link"/>
+    <origin xyz="0 0 ${third_link_length/2}" rpy="0 0 0"/>
+    <axis xyz="0 1 0"/>
+    <limit effort="10.0" velocity="1.0" lower="-1.57" upper="1.57"/>
+  </joint>
+  <joint name="joint5" type="revolute">
     <parent link="fourth_link"/>
-    <child link="gripper_base"/>
-    <origin xyz="0 0 ${fourth_link_length / 2}" rpy="0 0 0"/>
-  </joint>
-  <!-- Left Gripper Finger -->
-  <link name="left_finger">
-    <visual>
-      <geometry>
-        <box size="${gripper_finger_width} ${gripper_finger_length} ${gripper_finger_width}"/>
-      </geometry>
-      <material name="blue"/>
-    </visual>
-  </link>
-  <joint name="left_finger_joint" type="prismatic">
-    <parent link="gripper_base"/>
-    <child link="left_finger"/>
-    <origin xyz="0.05 0 ${gripper_finger_width / 2}" rpy="0 0 0"/>
+    <child link="gripper"/>
+    <origin xyz="0 0 ${fourth_link_length/2}" rpy="0 0 0"/>
     <axis xyz="0 1 0"/>
-    <limit lower="0" upper="${gripper_finger_range}" effort="10" velocity="0.05"/>
-  </joint>
-  <!-- Right Gripper Finger -->
-  <link name="right_finger">
-    <visual>
-      <geometry>
-        <box size="${gripper_finger_width} ${gripper_finger_length} ${gripper_finger_width}"/>
-      </geometry>
-      <material name="blue"/>
-    </visual>
-  </link>
-  <joint name="right_finger_joint" type="prismatic">
-    <parent link="gripper_base"/>
-    <child link="right_finger"/>
-    <origin xyz="-0.05 0 ${gripper_finger_width / 2}" rpy="0 0 0"/>
-    <axis xyz="0 -1 0"/>
-    <limit lower="0" upper="${gripper_finger_range}" effort="10" velocity="0.05"/>
+    <limit effort="10.0" velocity="1.0" lower="-1.57" upper="1.57"/>
   </joint>
 </robot>

Commit message: got the arm control working

File: src/sim_mdrs/urdf/arm.urdf.xacro (robot description, xacro)
@@ -1,13 +1,15 @@
 <?xml version="1.0"?>
 <robot xmlns:xacro="http://www.ros.org/wiki/xacro" name="my_robot_arm">
-  <plugin name="gazebo_ros_control" filename="libgazebo_ros_control.so">
-    <robotNamespace>/</robotNamespace>
-  </plugin>
+  <gazebo>
+    <plugin name="gazebo_ros2_control" filename="libgazebo_ros2_control.so">
+      <parameters>$(find sim_mdrs)/config/arm_control.yaml</parameters>
+    </plugin>
+  </gazebo>
   <!-- Properties -->
-  <xacro:property name="base_link_length" value="0.5"/>
-  <xacro:property name="first_link_length" value="0.5"/>
-  <xacro:property name="second_link_length" value="0.5"/>
-  <xacro:property name="third_link_length" value="0.5"/>
-  <xacro:property name="fourth_link_length" value="1.0"/>
+  <xacro:property name="base_height" value="0.0555"/>
+  <xacro:property name="B1_height" value="0.02"/>
+  <xacro:property name="B2_height" value="0.102"/>
+  <xacro:property name="arm_inf_height" value="0.228"/> <!-- will be 180 later-->
+  <xacro:property name="arm_sup_height" value="0.170"/>
   <xacro:property name="gripper_length" value="1.0"/>
   <xacro:property name="link_radius" value="0.05"/>
@@ -24,150 +26,198 @@
   </xacro:macro>
   <xacro:define_materials/>
+  <link name="world"></link>
+  <joint name="ground" type="fixed">
+    <parent link="world"/>
+    <child link="base_link"/>
+    <origin xyz="0 0 0.1" rpy="0 0 0"/>
+    <axis xyz="0 0 1"/>
+  </joint>
   <!-- Base Link -->
   <link name="base_link">
     <visual>
       <geometry>
-        <cylinder length="${base_link_length}" radius="${link_radius}"/>
+        <mesh filename="file://$(find sim_mdrs)/urdf/arm_meshes/B1.stl" scale="0.001 0.001 0.001"/>
       </geometry>
       <material name="gray"/>
-    </visual>
-    <collision>
-      <geometry>
-        <cylinder length="${base_link_length}" radius="${link_radius}"/>
-      </geometry>
-    </collision>
-    <inertial>
-      <mass value="1.0"/>
-      <origin xyz="0 0 0"/>
-      <inertia ixx="0.01" ixy="0.0" ixz="0.0" iyy="0.01" iyz="0.0" izz="0.01"/>
-    </inertial>
-  </link>
+      <origin xyz="0 -0.03 0.0" rpy="1.5708 0 3.14"/>
+    </visual>
+    <collision>
+      <geometry>
+        <mesh filename="file://$(find sim_mdrs)/urdf/arm_meshes/B1.stl" scale="0.001 0.001 0.001"/>
+      </geometry>
+      <origin xyz="0 -0.03 0" rpy="1.5708 0 3.14"/>
+    </collision>
+  </link>
+  <joint name="joint1" type="fixed">
+    <parent link="base_link"/>
+    <child link="B1_fixe"/>
+    <origin xyz="0 0 0" rpy="0 0 0"/>
+    <axis xyz="0 0 1"/>
+  </joint>
   <!-- First Link -->
-  <link name="first_link">
-    <visual>
-      <geometry>
-        <cylinder length="${first_link_length}" radius="${link_radius}"/>
+  <link name="B1_fixe">
+    <visual>
+      <geometry>
+        <mesh filename="file://$(find sim_mdrs)/urdf/arm_meshes/B1_fixe2.stl" scale="0.001 0.001 0.001"/>
       </geometry>
       <material name="blue"/>
-    </visual>
-    <collision>
-      <geometry>
-        <cylinder length="${first_link_length}" radius="${link_radius}"/>
-      </geometry>
-    </collision>
-    <inertial>
-      <mass value="0.5"/>
-      <origin xyz="0 0 0"/>
-      <inertia ixx="0.005" ixy="0.0" ixz="0.0" iyy="0.005" iyz="0.0" izz="0.005"/>
-    </inertial>
-  </link>
-<joint name="joint2" type="revolute">
-    <parent link="first_link"/>
-    <child link="second_link"/>
-    <origin xyz="0 0 ${second_link_length / 2}" rpy="0 0 0"/>
+      <origin xyz="0 0 ${base_height}" rpy="1.5708 0 0"/>
+    </visual>
+    <collision>
+      <geometry>
+        <mesh filename="file://$(find sim_mdrs)/urdf/arm_meshes/B1_fixe2.stl" scale="0.001 0.001 0.001"/>
+      </geometry>
+      <origin xyz="0 0 ${base_height}" rpy="1.5708 0 0"/>
+    </collision>
+    <inertial>
+      <mass value="0.01"/>
+      <origin xyz="0 0 0"/>
+      <inertia ixx="0.0001" ixy="0.0" ixz="0.0" iyy="0.0001" iyz="0.0" izz="0.0001"/>
+    </inertial>
+  </link>
+  <joint name="joint2" type="revolute">
+    <parent link="B1_fixe"/>
+    <child link="B2"/>
+    <origin xyz="0 0 0" rpy="0 0 0"/>
+    <axis xyz="0 0 1"/>
+    <limit lower="-1.57" upper="1.57" effort="10" velocity="1"/>
+  </joint>
+  <link name="B2">
+    <visual>
+      <geometry>
+        <mesh filename="file://$(find sim_mdrs)/urdf/arm_meshes/B2.stl" scale="0.001 0.001 0.001"/>
+      </geometry>
+      <material name="red"/>
+      <origin xyz="0 0 ${B1_height}" rpy="1.5708 0 0"/>
+    </visual>
+    <collision>
+      <geometry>
+        <mesh filename="file://$(find sim_mdrs)/urdf/arm_meshes/B2.stl" scale="0.001 0.001 0.001"/>
+      </geometry>
+      <origin xyz="0 0 ${B1_height}" rpy="1.5708 0 0"/>
+    </collision>
+    <inertial>
+      <mass value="0.1"/>
+      <origin xyz="0 0 0"/>
+      <inertia ixx="0.0001" ixy="0.0" ixz="0.0" iyy="0.0001" iyz="0.0" izz="0.000001"/>
+    </inertial>
+  </link>
+  <joint name="joint3" type="revolute">
+    <parent link="B2"/>
+    <child link="arm_inf"/>
+    <origin xyz="0 0 ${B2_height}" rpy="0 0 0"/>
     <axis xyz="1 0 0"/>
     <limit lower="-1.57" upper="1.57" effort="10" velocity="1"/>
   </joint>
-  <link name="second_link">
-    <visual>
-      <geometry>
-        <cylinder length="${second_link_length}" radius="${link_radius}"/>
-      </geometry>
-      <material name="red"/>
-    </visual>
-    <collision>
-      <geometry>
-        <cylinder length="${second_link_length}" radius="${link_radius}"/>
-      </geometry>
-    </collision>
-    <inertial>
-      <mass value="0.5"/>
-      <origin xyz="0 0 0"/>
-      <inertia ixx="0.005" ixy="0.0" ixz="0.0" iyy="0.005" iyz="0.0" izz="0.005"/>
-    </inertial>
-  </link>
-<joint name="joint3" type="revolute">
-    <parent link="second_link"/>
-    <child link="third_link"/>
-    <origin xyz="0 0 ${third_link_length / 2}" rpy="0 0 0"/>
+  <link name="arm_inf">
+    <visual>
+      <geometry>
+        <mesh filename="file://$(find sim_mdrs)/urdf/arm_meshes/arm_inf.stl" scale="0.001 0.001 0.001"/>
+      </geometry>
+      <material name="blue"/>
+     <origin xyz="0.02 -0.02 ${2*arm_inf_height/3}" rpy="0 1.5708 0"/>
+    </visual>
+    <collision>
+      <geometry>
+        <mesh filename="file://$(find sim_mdrs)/urdf/arm_meshes/arm_inf.stl" scale="0.001 0.001 0.001"/>
+      </geometry>
+      <origin xyz="0.02 -0.02 ${2*arm_inf_height/3}" rpy="0 1.5708 0"/>
+    </collision>
+    <inertial>
+      <mass value="0.1"/>
+      <origin xyz="0 0 0"/>
+      <inertia ixx="0.0001" ixy="0.0" ixz="0.0" iyy="0.0001" iyz="0.0" izz="0.0001"/>
+    </inertial>
+  </link>
+  <joint name="joint4" type="revolute">
+    <parent link="arm_inf"/>
+    <child link="arm_sup"/>
+    <origin xyz="0 0 ${arm_inf_height-0.02}" rpy="0 0 0"/>
     <axis xyz="1 0 0"/>
     <limit lower="-1.57" upper="1.57" effort="10" velocity="1"/>
   </joint>
-  <link name="third_link">
-    <visual>
-      <geometry>
-        <cylinder length="${third_link_length}" radius="${link_radius}"/>
-      </geometry>
-      <material name="blue"/>
-    </visual>
-    <collision>
-      <geometry>
-        <cylinder length="${third_link_length}" radius="${link_radius}"/>
-      </geometry>
-    </collision>
-    <inertial>
-      <mass value="0.5"/>
-      <origin xyz="0 0 0"/>
-      <inertia ixx="0.005" ixy="0.0" ixz="0.0" iyy="0.005" iyz="0.0" izz="0.005"/>
-    </inertial>
-  </link>
-<joint name="joint4" type="revolute">
-    <parent link="third_link"/>
-    <child link="arm_link"/>
-    <origin xyz="0 0 ${base_link_length / 2}" rpy="0 0 0"/>
+  <link name="arm_sup">
+    <visual>
+      <geometry>
+        <mesh filename="file://$(find sim_mdrs)/urdf/arm_meshes/arm_sup.stl" scale="0.001 0.001 0.001"/>
+      </geometry>
+      <material name="red"/>
+      <origin xyz="0.035 -0.02 -0.03" rpy="1.5708 1.5708 1.5708"/>
+    </visual>
+    <collision>
+      <geometry>
+        <mesh filename="file://$(find sim_mdrs)/urdf/arm_meshes/arm_sup.stl" scale="0.001 0.001 0.001"/>
+      </geometry>
+      <origin xyz="0.035 -0.02 -0.03" rpy="1.5708 1.5708 1.5708"/>
+    </collision>
+    <inertial>
+      <mass value="0.2"/>
+      <origin xyz="0 0 0"/>
+      <inertia ixx="0.0001" ixy="0.0" ixz="0.0" iyy="0.0001" iyz="0.0" izz="0.0001"/>
+    </inertial>
+  </link>
+  <joint name="joint5" type="revolute">
+    <parent link="arm_sup"/>
+    <child link="gripper"/>
+    <origin xyz="0 0 ${arm_sup_height}" rpy="0 0 0"/>
     <axis xyz="1 0 0"/>
-    <limit lower="-1.57" upper="1.57" effort="10" velocity="1"/>
-  </joint>
-  <link name="arm_link">
-    <visual>
-      <geometry>
-        <cylinder length="${fourth_link_length}" radius="${link_radius}"/>
-      </geometry>
-      <material name="red"/>
-    </visual>
-    <collision>
-      <geometry>
-        <cylinder length="${fourth_link_length}" radius="${link_radius}"/>
-      </geometry>
-    </collision>
-    <inertial>
-      <mass value="0.8"/>
-      <origin xyz="0 0 0"/>
-      <inertia ixx="0.01" ixy="0.0" ixz="0.0" iyy="0.01" iyz="0.0" izz="0.01"/>
-    </inertial>
-  </link>
-  <!-- Gripper Link -->
+    <limit effort="10.0" velocity="1.0" lower="-1.57" upper="1.57"/>
+  </joint>
   <link name="gripper">
     <visual>
       <geometry>
-        <cylinder length="${gripper_length}" radius="${link_radius}"/>
+        <mesh filename="file://$(find sim_mdrs)/urdf/arm_meshes/jonc_pliers.stl" scale="0.001 0.001 0.001"/>
       </geometry>
       <material name="gray"/>
-    </visual>
-  </link>
-  <joint name="gripper_joint" type="fixed">
-    <parent link="arm_link"/>
-    <child link="gripper_base"/>
-    <origin xyz="0 0 ${fourth_link_length / 2}" rpy="0 0 0"/>
-  </joint>
-  <!-- Left Gripper Finger -->
-  <link name="left_finger">
-    <visual>
-      <geometry>
-        <cylinder length="${gripper_length}" radius="${link_radius}"/>
-      </geometry>
-    </collision>
-    <inertial>
-      <mass value="0.3"/>
-      <origin xyz="0 0 0"/>
-      <inertia ixx="0.002" ixy="0.0" ixz="0.0" iyy="0.002" iyz="0.0" izz="0.002"/>
-    </inertial>
-  </link>
-  <joint name="joint5" type="revolute">
-    <parent link="fourth_link"/>
-    <child link="gripper"/>
-    <origin xyz="0 0 ${fourth_link_length/2}" rpy="0 0 0"/>
-    <axis xyz="0 1 0"/>
-    <limit effort="10.0" velocity="1.0" lower="-1.57" upper="1.57"/>
-  </joint>
+      <origin xyz="0.04 -0.02 -0.02" rpy="0 1.5708 0"/>
+    </visual>
+    <collision>
+      <geometry>
+        <mesh filename="file://$(find sim_mdrs)/urdf/arm_meshes/jonc_pliers.stl" scale="0.001 0.001 0.001"/>
+      </geometry>
+      <origin xyz="0.04 -0.02 -0.02" rpy="0 1.5708 0"/>
+    </collision>
+    <inertial>
+      <mass value="0.2"/>
+      <origin xyz="0 0 0"/>
+      <inertia ixx="0.0001" ixy="0.0" ixz="0.0" iyy="0.0001" iyz="0.0" izz="0.0001"/>
+    </inertial>
+  </link>
+  <transmission name="joint2_transmission">
+    <type>transmission_interface/SimpleTransmission</type>
+    <joint name="joint2">
+      <hardwareInterface>hardware_interface/PositionJointInterface</hardwareInterface>
+    </joint>
+    <actuator name="joint2_motor">
+      <mechanicalReduction>1</mechanicalReduction>
+    </actuator>
+  </transmission>
+  <transmission name="joint3_transmission">
+    <type>transmission_interface/SimpleTransmission</type>
+    <joint name="joint3">
+      <hardwareInterface>hardware_interface/PositionJointInterface</hardwareInterface>
+    </joint>
+    <actuator name="joint3_motor">
+      <mechanicalReduction>1</mechanicalReduction>
+    </actuator>
+  </transmission>
+  <transmission name="joint4_transmission">
+    <type>transmission_interface/SimpleTransmission</type>
+    <joint name="joint4">
+      <hardwareInterface>hardware_interface/PositionJointInterface</hardwareInterface>
+    </joint>
+    <actuator name="joint4_motor">
+      <mechanicalReduction>1</mechanicalReduction>
+    </actuator>
+  </transmission>
+  <transmission name="joint5_transmission">
+    <type>transmission_interface/SimpleTransmission</type>
+    <joint name="joint5">
+      <hardwareInterface>hardware_interface/PositionJointInterface</hardwareInterface>
+    </joint>
+    <actuator name="joint5_motor">
+      <mechanicalReduction>1</mechanicalReduction>
+    </actuator>
+  </transmission>
+  <xacro:include filename="$(find sim_mdrs)/urdf/arm_control.urdf.xacro"/>
 </robot>
